File: kicad/SmartPendant.kicad_pcb (KiCad board)
At the start: 2 copper layers, 125 x 59 mm, 50 parts, among them J1 UART, J2 ST-LINK, J3 Encoder, J5 Display, J6 USB_C_Receptacle_USB2.0_16P, J8 Micro_SD_Card_Det1, Q1 MMBT3904, U1 WEACT BLACKPILL F4X1, U2 AMS1117-3.3, U3 MB85RC256VPNF-G-JNERE1

Commit message: Fix positioning issues.
Parts:
- moved D2 32.8 mm to (218.8, 86.5), turned to 0 degrees
- moved U2 28.6 mm to (216.7, 62.1)
- moved BTN_USR1 1.40 mm to (245.1, 99.0)
- moved R13 1.22 mm to (245.6, 93.9)
- moved J6 0.51 mm to (246.1, 78.0)
- moved BTN_LD1 0.50 mm to (197.9, 52.9)
- moved BTN_LU1 0.50 mm to (213.0, 52.9)
- moved BTN_RD1 0.50 mm to (197.9, 102.1)
- moved BTN_RU1 0.50 mm to (213.0, 102.1)
- moved R4 0.41 mm to (239.7, 76.3)
- moved R3 0.36 mm to (239.8, 79.2)
- moved D1 0.20 mm to (238.8, 81.8)
Other:
- outline, holes or cut-outs redrawn
Changed lines of the file:
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@@
 	(footprint "Custom:SMD_Push_Side_button_3x6x3.5mm"
 		(layer "F.Cu")
-		(at 198.4 52.9 180)
+		(at 197.9 52.9 180)
 		(descr "Microminiature SMT Side Actuated, 4.2 x 2.8 x 1.42mm with pegs, https://www.ckswitches.com/media/1482/kms.pdf")
 		(tags "Switch SPST KMS2")
@@
 	(footprint "PCM_Resistor_SMD_AKL:R_0603_1608Metric"
 		(layer "F.Cu")
-		(at 239.713 75.8444 180)
+		(at 239.6998 76.2508 180)
 		(descr "Resistor SMD 0603 (1608 Metric), square (rectangular) end terminal, IPC_7351 nominal, (Body size source: IPC-SM-782 page 72, https://www.pcb-3d.com/wordpress/wp-content/uploads/ipc-sm-782a_amendment_1_and_2.pdf), Alternate KiCad Library")
 		(tags "resistor")
@@
 	(footprint "Custom:USB_C_Receptacle_AliExpress_16pin"
 		(layer "F.Cu")
-		(at 246.1166 77.4916 90)
+		(at 246.1166 78 90)
 		(descr "USB Type C, right-angle, SMT, https://datasheet.lcsc.com/szlcsc/1811141824_XKB-Enterprise-U262-161N-4BVC11_C319148.pdf")
 		(tags "USB C Type-C Receptacle SMD")
@@
 	(footprint "Custom:SMD_Push_Side_button_3x6x3.5mm"
 		(layer "F.Cu")
-		(at 198.4 102.1)
+		(at 197.9 102.1)
 		(descr "Microminiature SMT Side Actuated, 4.2 x 2.8 x 1.42mm with pegs, https://www.ckswitches.com/media/1482/kms.pdf")
 		(tags "Switch SPST KMS2")
@@
 	(footprint "PCM_Resistor_SMD_AKL:R_0603_1608Metric"
 		(layer "F.Cu")
-		(at 245.618 95.1484)
+		(at 245.618 93.9292)
 		(descr "Resistor SMD 0603 (1608 Metric), square (rectangular) end terminal, IPC_7351 nominal, (Body size source: IPC-SM-782 page 72, https://www.pcb-3d.com/wordpress/wp-content/uploads/ipc-sm-782a_amendment_1_and_2.pdf), Alternate KiCad Library")
 		(tags "resistor")
 		(property "Reference" "R13"
-			(at -0.0254 -1.8034 180)
+			(at -0.8636 -2.5654 270)
 			(layer "F.SilkS")
 			(effects
@@
 	(footprint "PCM_Diode_SMD_AKL:D_SOD-123"
 		(layer "F.Cu")
-		(at 238.8372 81.6102)
+		(at 238.8372 81.8134)
 		(descr "SOD-123, Alternate KiCad Library")
 		(tags "SOD-123")
 		(property "Reference" "D1"
-			(at -3.7348 0.3302 0)
+			(at 1.1674 2.5146 0)
 			(layer "F.SilkS")
 			(effects
@@
 	(footprint "PCM_Diode_SMD_AKL:D_SOD-123"
 		(layer "F.Cu")
-		(at 245.4656 67.4624 -90)
+		(at 218.7702 86.4616)
 		(descr "SOD-123, Alternate KiCad Library")
 		(tags "SOD-123")
 		(property "Reference" "D2"
-			(at 0.889 -2.127 90)
+			(at 3.8354 0.127 0)
 			(layer "F.SilkS")
 			(effects
@@
 		)
 		(property "Value" "1N5819"
-			(at 0 2.1 90)
+			(at 0 2.1 0)
 			(layer "F.Fab")
 			(hide yes)
@@
 		)
 		(property "Datasheet" "~"
-			(at 0 0 90)
+			(at 0 0 0)
 			(layer "F.Fab")
 			(hide yes)
@@
 		)
 		(property "Description" "Schottky diode"
-			(at 0 0 90)
+			(at 0 0 0)
 			(layer "F.Fab")
 			(hide yes)
@@
 		(attr smd)
 		(fp_line
-			(start -2.4 1.2)
-			(end 2.4 1.2)
+			(start -2.4 -1.2)
+			(end -2.4 1.2)
 			(stroke
 				(width 0.12)
@@
 		)
 		(fp_line
-			(start 2.4 1.2)
-			(end 2.4 -1.2)
+			(start -2.4 1.2)
+			(end 2.4 1.2)
 			(stroke
 				(width 0.12)
@@
 		)
 		(fp_line
-			(start -2.4 -1.2)
-			(end -2.4 1.2)
+			(start 2.4 -1.2)
+			(end -2.4 -1.2)
 			(stroke
 				(width 0.12)
@@
 		)
 		(fp_line
-			(start 2.4 -1.2)
-			(end -2.4 -1.2)
+			(start 2.4 1.2)
+			(end 2.4 -1.2)
 			(stroke
 				(width 0.12)
@@
 		(fp_poly
 			(pts
-				(xy -0.6 1.5) (xy -1.4 1.5) (xy -1.4 1.2) (xy -0.6 1.2)
+				(xy -0.6 -1.2) (xy -1.4 -1.2) (xy -1.4 -1.5) (xy -0.6 -1.5)
 			)
 			(stroke
@@
 		(fp_poly
 			(pts
-				(xy -0.6 -1.2) (xy -1.4 -1.2) (xy -1.4 -1.5) (xy -0.6 -1.5)
+				(xy -0.6 1.5) (xy -1.4 1.5) (xy -1.4 1.2) (xy -0.6 1.2)
 			)
 			(stroke
@@
 		)
 		(fp_line
-			(start 2.35 1.15)
+			(start -2.35 -1.15)
 			(end -2.35 1.15)
 			(stroke
@@
 		(fp_line
 			(start -2.35 -1.15)
-			(end -2.35 1.15)
+			(end 2.35 -1.15)
 			(stroke
 				(width 0.05)
@@
 		)
 		(fp_line
-			(start -2.35 -1.15)
-			(end 2.35 -1.15)
+			(start 2.35 -1.15)
+			(end 2.35 1.15)
 			(stroke
 				(width 0.05)
@@
 		)
 		(fp_line
-			(start 2.35 -1.15)
-			(end 2.35 1.15)
+			(start 2.35 1.15)
+			(end -2.35 1.15)
 			(stroke
 				(width 0.05)
@@
 		)
 		(fp_line
-			(start -1.4 0.9)
-			(end -1.4 -0.9)
+			(start -1.9 -0.3)
+			(end -1.9 0.3)
 			(stroke
 				(width 0.1)
@@
 		)
 		(fp_line
-			(start 1.4 0.9)
-			(end -1.4 0.9)
+			(start -1.9 0.3)
+			(end -1.4 0.3)
 			(stroke
 				(width 0.1)
@@
 		)
 		(fp_line
-			(start -1.9 0.3)
-			(end -1.4 0.3)
+			(start -1.4 -0.9)
+			(end 1.4 -0.9)
 			(stroke
 				(width 0.1)
@@
 		)
 		(fp_line
-			(start 1.5 0.3)
-			(end 1.4 0.3)
+			(start -1.4 -0.3)
+			(end -1.9 -0.3)
 			(stroke
 				(width 0.1)
@@
 		)
 		(fp_line
-			(start 1.9 0.3)
-			(end 1.5 0.3)
+			(start -1.4 0.9)
+			(end -1.4 -0.9)
 			(stroke
 				(width 0.1)
@@
 		)
 		(fp_line
-			(start -1.9 -0.3)
-			(end -1.9 0.3)
+			(start 1.4 -0.9)
+			(end 1.4 0.9)
 			(stroke
 				(width 0.1)
@@
 		)
 		(fp_line
-			(start -1.4 -0.3)
-			(end -1.9 -0.3)
+			(start 1.4 -0.3)
+			(end 1.9 -0.3)
 			(stroke
 				(width 0.1)
@@
 		)
 		(fp_line
-			(start 1.4 -0.3)
-			(end 1.9 -0.3)
+			(start 1.4 0.9)
+			(end -1.4 0.9)
 			(stroke
 				(width 0.1)
@@
 		)
 		(fp_line
-			(start 1.9 -0.3)
-			(end 1.9 0.3)
+			(start 1.5 0.3)
+			(end 1.4 0.3)
 			(stroke
 				(width 0.1)
@@
 		)
 		(fp_line
-			(start -1.4 -0.9)
-			(end 1.4 -0.9)
+			(start 1.9 -0.3)
+			(end 1.9 0.3)
 			(stroke
 				(width 0.1)
@@
 		)
 		(fp_line
-			(start 1.4 -0.9)
-			(end 1.4 0.9)
+			(start 1.9 0.3)
+			(end 1.5 0.3)
 			(stroke
 				(width 0.1)
@@
 		)
 		(fp_text user "${REFERENCE}"
-			(at 0.4 0 90)
+			(at 0.4 0 0)
 			(layer "F.Fab")
 			(effects
@@
 		)
 		(pad "1" smd roundrect
-			(at -1.65 0 270)
+			(at -1.65 0)
 			(size 0.9 1.2)
 			(layers "F.Cu" "F.Mask" "F.Paste")
@@
 		)
 		(pad "2" smd roundrect
-			(at 1.65 0 270)
+			(at 1.65 0)
 			(size 0.9 1.2)
 			(layers "F.Cu" "F.Mask" "F.Paste")
@@
 	(footprint "Custom:SMD_Push_Side_button_3x6x3.5mm"
 		(layer "F.Cu")
-		(at 213.5 102.1)
+		(at 213 102.1)
 		(descr "Microminiature SMT Side Actuated, 4.2 x 2.8 x 1.42mm with pegs, https://www.ckswitches.com/media/1482/kms.pdf")
 		(tags "Switch SPST KMS2")
@@
 	(footprint "Custom:SMD_Push_Side_button_3x6x3.5mm"
 		(layer "F.Cu")
-		(at 245.0798 100.4 90)
+		(at 245.0798 99 90)
 		(descr "Microminiature SMT Side Actuated, 4.2 x 2.8 x 1.42mm with pegs, https://www.ckswitches.com/media/1482/kms.pdf")
 		(tags "Switch SPST KMS2")
@@
 	(footprint "PCM_Package_TO_SOT_SMD_AKL:SOT-223-3_TabPin2"
 		(layer "F.Cu")
-		(at 245.1604 59.5376)
+		(at 216.6874 62.0522)
 		(descr "module CMS SOT223 4 pins, Alternate KiCad Library")
 		(tags "CMS SOT")
@@
 	(footprint "Custom:SMD_Push_Side_button_3x6x3.5mm"
 		(layer "F.Cu")
-		(at 213.5 52.9 180)
+		(at 213 52.9 180)
 		(descr "Microminiature SMT Side Actuated, 4.2 x 2.8 x 1.42mm with pegs, https://www.ckswitches.com/media/1482/kms.pdf")
 		(tags "Switch SPST KMS2")
@@
 	(footprint "PCM_Resistor_SMD_AKL:R_0603_1608Metric"
 		(layer "F.Cu")
-		(at 239.7506 78.8924 180)
+		(at 239.7506 79.248 180)
 		(descr "Resistor SMD 0603 (1608 Metric), square (rectangular) end terminal, IPC_7351 nominal, (Body size source: IPC-SM-782 page 72, https://www.pcb-3d.com/wordpress/wp-content/uploads/ipc-sm-782a_amendment_1_and_2.pdf), Alternate KiCad Library")
 		(tags "resistor")
@@
 	)
 	(gr_line
+		(start 246 87)
+		(end 246 92)
+		(stroke
+			(width 0.05)
+			(type solid)
+		)
+		(layer "Edge.Cuts")
+	)
+	(gr_arc
+		(start 250 83)
+		(mid 248.828427 85.828427)
+		(end 246 87)
+		(stroke
+			(width 0.05)
+			(type solid)
+		)
+		(layer "Edge.Cuts")
+	)
+	(gr_line
+		(start 248 94)
+		(end 248 107)
+		(stroke
+			(width 0.05)
+			(type solid)
+		)
+		(layer "Edge.Cuts")
+	)
+	(gr_arc
+		(start 250 54)
+		(mid 248.828427 56.828427)
+		(end 246 58)
+		(stroke
+			(width 0.05)
+			(type solid)
+		)
+		(layer "Edge.Cuts")
+	)
+	(gr_line
+		(start 250 72)
+		(end 250 83)
+		(stroke
+			(width 0.05)
+			(type solid)
+		)
+		(layer "Edge.Cuts")
+	)
+	(gr_line
 		(start 245 48)
 		(end 250 48)
@@
 	(gr_line
 		(start 250 48)
-		(end 250 107)
+		(end 250 54)
 		(stroke
 			(width 0.049999)
@@
 	(gr_curve
 		(pts
-			(xy 141.999998 77.50008) (xy 141.698479 95.310577) (xy 125 99.000004) (xy 125 99.000004)
+			(xy 141.999998 77.50008) (xy 141.698479 95.310577) (xy 125 99.000004) (xy 125 99)
 		)
 		(stroke
@@
 	(gr_line
 		(start 245 107)
-		(end 250 107)
+		(end 248 107)
 		(stroke
 			(width 0.05)
@@
 		(layer "Edge.Cuts")
 	)
+	(gr_arc
+		(start 246 92)
+		(mid 247.414214 92.585786)
+		(end 248 94)
+		(stroke
+			(width 0.05)
+			(type solid)
+		)
+		(layer "Edge.Cuts")
+	)
+	(gr_arc
+		(start 246 68)
+		(mid 248.828427 69.171573)
+		(end 250 72)
+		(stroke
+			(width 0.05)
+			(type solid)
+		)
+		(layer "Edge.Cuts")
+	)
 	(gr_curve
 		(pts
@@
 		)
 		(layer "Edge.Cuts")
+	)
+	(gr_line
+		(start 246 58)
+		(end 246 68)
+		(stroke
+			(width 0.05)
+			(type default)
+		)
+		(layer "Edge.Cuts")
